File: Front/MIDI_Tangle_Front.sch (KiCad schematic (older format))
At the start: 28 parts, among them J1 Screw_Terminal_01x01, J10 Screw_Terminal_01x01, J11 Screw_Terminal_01x01, J12 Screw_Terminal_01x01, J13 Screw_Terminal_01x01, J14 Screw_Terminal_01x01, J15 Screw_Terminal_01x01, J16 Screw_Terminal_01x01, J17 Screw_Terminal_01x01, J18 Screw_Terminal_01x01, J19 Screw_Terminal_01x01, J2 Screw_Terminal_01x01, J20 Screw_Terminal_01x01, J3 Screw_Terminal_01x01, J4 Screw_Terminal_01x01, J5 Screw_Terminal_01x01, J6 Screw_Terminal_01x01, J7 Screw_Terminal_01x01, J8 Screw_Terminal_01x01, J9 Screw_Terminal_01x01

Commit message: Add custom footprints and symbols
Parts:
- H1, H2, H3, H4, H5, H6, H7, H8: footprint CustomLib:TactileHole -> Custom_FP:TactileHole
- J1, J2, J3, J4: footprint CustomLib:Wide_M3 -> Custom_FP:Wide_M3
- J10, J11, J12, J13, J14, J15, J16, J17, J18, J19, J20, J5, J6, J7, J8, J9: footprint MountingHole:MountingHole_6.2mm_M6 -> Custom_FP:MountingHole_PJ398SM
Changed lines of the file:
@@
 F 0 "J5" H 5980 1992 50  0000 L CNN
 F 1 "Screw_Terminal_01x01" H 5980 1901 50  0000 L CNN
-F 2 "MountingHole:MountingHole_6.2mm_M6" H 5900 1950 50  0001 C CNN
+F 2 "Custom_FP:MountingHole_PJ398SM" H 5900 1950 50  0001 C CNN
 F 3 "~" H 5900 1950 50  0001 C CNN
 	1    5900 1950
@@
 F 0 "J6" H 5980 2192 50  0000 L CNN
 F 1 "Screw_Terminal_01x01" H 5980 2101 50  0000 L CNN
-F 2 "MountingHole:MountingHole_6.2mm_M6" H 5900 2150 50  0001 C CNN
+F 2 "Custom_FP:MountingHole_PJ398SM" H 5900 2150 50  0001 C CNN
 F 3 "~" H 5900 2150 50  0001 C CNN
 	1    5900 2150
@@
 F 0 "J7" H 5980 2392 50  0000 L CNN
 F 1 "Screw_Terminal_01x01" H 5980 2301 50  0000 L CNN
-F 2 "MountingHole:MountingHole_6.2mm_M6" H 5900 2350 50  0001 C CNN
+F 2 "Custom_FP:MountingHole_PJ398SM" H 5900 2350 50  0001 C CNN
 F 3 "~" H 5900 2350 50  0001 C CNN
 	1    5900 2350
@@
 F 0 "J8" H 5980 2592 50  0000 L CNN
 F 1 "Screw_Terminal_01x01" H 5980 2501 50  0000 L CNN
-F 2 "MountingHole:MountingHole_6.2mm_M6" H 5900 2550 50  0001 C CNN
+F 2 "Custom_FP:MountingHole_PJ398SM" H 5900 2550 50  0001 C CNN
 F 3 "~" H 5900 2550 50  0001 C CNN
 	1    5900 2550
@@
 F 0 "J9" H 5980 2792 50  0000 L CNN
 F 1 "Screw_Terminal_01x01" H 5980 2701 50  0000 L CNN
-F 2 "MountingHole:MountingHole_6.2mm_M6" H 5900 2750 50  0001 C CNN
+F 2 "Custom_FP:MountingHole_PJ398SM" H 5900 2750 50  0001 C CNN
 F 3 "~" H 5900 2750 50  0001 C CNN
 	1    5900 2750
@@
 F 0 "J10" H 5980 2992 50  0000 L CNN
 F 1 "Screw_Terminal_01x01" H 5980 2901 50  0000 L CNN
-F 2 "MountingHole:MountingHole_6.2mm_M6" H 5900 2950 50  0001 C CNN
+F 2 "Custom_FP:MountingHole_PJ398SM" H 5900 2950 50  0001 C CNN
 F 3 "~" H 5900 2950 50  0001 C CNN
 	1    5900 2950
@@
 F 0 "J11" H 5980 3192 50  0000 L CNN
 F 1 "Screw_Terminal_01x01" H 5980 3101 50  0000 L CNN
-F 2 "MountingHole:MountingHole_6.2mm_M6" H 5900 3150 50  0001 C CNN
+F 2 "Custom_FP:MountingHole_PJ398SM" H 5900 3150 50  0001 C CNN
 F 3 "~" H 5900 3150 50  0001 C CNN
 	1    5900 3150
@@
 F 0 "J12" H 5980 3392 50  0000 L CNN
 F 1 "Screw_Terminal_01x01" H 5980 3301 50  0000 L CNN
-F 2 "MountingHole:MountingHole_6.2mm_M6" H 5900 3350 50  0001 C CNN
+F 2 "Custom_FP:MountingHole_PJ398SM" H 5900 3350 50  0001 C CNN
 F 3 "~" H 5900 3350 50  0001 C CNN
 	1    5900 3350
@@
 F 0 "J13" H 5980 3592 50  0000 L CNN
 F 1 "Screw_Terminal_01x01" H 5980 3501 50  0000 L CNN
-F 2 "MountingHole:MountingHole_6.2mm_M6" H 5900 3550 50  0001 C CNN
+F 2 "Custom_FP:MountingHole_PJ398SM" H 5900 3550 50  0001 C CNN
 F 3 "~" H 5900 3550 50  0001 C CNN
 	1    5900 3550
@@
 F 0 "J14" H 5980 3792 50  0000 L CNN
 F 1 "Screw_Terminal_01x01" H 5980 3701 50  0000 L CNN
-F 2 "MountingHole:MountingHole_6.2mm_M6" H 5900 3750 50  0001 C CNN
+F 2 "Custom_FP:MountingHole_PJ398SM" H 5900 3750 50  0001 C CNN
 F 3 "~" H 5900 3750 50  0001 C CNN
 	1    5900 3750
@@
 F 0 "J15" H 5980 3992 50  0000 L CNN
 F 1 "Screw_Terminal_01x01" H 5980 3901 50  0000 L CNN
-F 2 "MountingHole:MountingHole_6.2mm_M6" H 5900 3950 50  0001 C CNN
+F 2 "Custom_FP:MountingHole_PJ398SM" H 5900 3950 50  0001 C CNN
 F 3 "~" H 5900 3950 50  0001 C CNN
 	1    5900 3950
@@
 F 0 "J16" H 5980 4192 50  0000 L CNN
 F 1 "Screw_Terminal_01x01" H 5980 4101 50  0000 L CNN
-F 2 "MountingHole:MountingHole_6.2mm_M6" H 5900 4150 50  0001 C CNN
+F 2 "Custom_FP:MountingHole_PJ398SM" H 5900 4150 50  0001 C CNN
 F 3 "~" H 5900 4150 50  0001 C CNN
 	1    5900 4150
@@
 F 0 "J17" H 5980 4392 50  0000 L CNN
 F 1 "Screw_Terminal_01x01" H 5980 4301 50  0000 L CNN
-F 2 "MountingHole:MountingHole_6.2mm_M6" H 5900 4350 50  0001 C CNN
+F 2 "Custom_FP:MountingHole_PJ398SM" H 5900 4350 50  0001 C CNN
 F 3 "~" H 5900 4350 50  0001 C CNN
 	1    5900 4350
@@
 F 0 "J18" H 5980 4592 50  0000 L CNN
 F 1 "Screw_Terminal_01x01" H 5980 4501 50  0000 L CNN
-F 2 "MountingHole:MountingHole_6.2mm_M6" H 5900 4550 50  0001 C CNN
+F 2 "Custom_FP:MountingHole_PJ398SM" H 5900 4550 50  0001 C CNN
 F 3 "~" H 5900 4550 50  0001 C CNN
 	1    5900 4550
@@
 F 0 "J19" H 5980 4792 50  0000 L CNN
 F 1 "Screw_Terminal_01x01" H 5980 4701 50  0000 L CNN
-F 2 "MountingHole:MountingHole_6.2mm_M6" H 5900 4750 50  0001 C CNN
+F 2 "Custom_FP:MountingHole_PJ398SM" H 5900 4750 50  0001 C CNN
 F 3 "~" H 5900 4750 50  0001 C CNN
 	1    5900 4750
@@
 F 0 "J20" H 5980 4992 50  0000 L CNN
 F 1 "Screw_Terminal_01x01" H 5980 4901 50  0000 L CNN
-F 2 "MountingHole:MountingHole_6.2mm_M6" H 5900 4950 50  0001 C CNN
+F 2 "Custom_FP:MountingHole_PJ398SM" H 5900 4950 50  0001 C CNN
 F 3 "~" H 5900 4950 50  0001 C CNN
 	1    5900 4950
@@
 F 0 "J1" H 4480 1992 50  0000 L CNN
 F 1 "Screw_Terminal_01x01" H 4480 1901 50  0000 L CNN
-F 2 "CustomLib:Wide_M3" H 4400 1950 50  0001 C CNN
+F 2 "Custom_FP:Wide_M3" H 4400 1950 50  0001 C CNN
 F 3 "~" H 4400 1950 50  0001 C CNN
 	1    4400 1950
@@
 F 0 "J2" H 4480 2242 50  0000 L CNN
 F 1 "Screw_Terminal_01x01" H 4480 2151 50  0000 L CNN
-F 2 "CustomLib:Wide_M3" H 4400 2200 50  0001 C CNN
+F 2 "Custom_FP:Wide_M3" H 4400 2200 50  0001 C CNN
 F 3 "~" H 4400 2200 50  0001 C CNN
 	1    4400 2200
@@
 F 0 "J3" H 4480 2492 50  0000 L CNN
 F 1 "Screw_Terminal_01x01" H 4480 2401 50  0000 L CNN
-F 2 "CustomLib:Wide_M3" H 4400 2450 50  0001 C CNN
+F 2 "Custom_FP:Wide_M3" H 4400 2450 50  0001 C CNN
 F 3 "~" H 4400 2450 50  0001 C CNN
 	1    4400 2450
@@
 F 0 "J4" H 4480 2742 50  0000 L CNN
 F 1 "Screw_Terminal_01x01" H 4480 2651 50  0000 L CNN
-F 2 "CustomLib:Wide_M3" H 4400 2700 50  0001 C CNN
+F 2 "Custom_FP:Wide_M3" H 4400 2700 50  0001 C CNN
 F 3 "~" H 4400 2700 50  0001 C CNN
 	1    4400 2700
@@
 F 0 "H3" H 2850 1946 50  0000 L CNN
 F 1 "MountingHole" H 2850 1855 50  0000 L CNN
-F 2 "CustomLib:TactileHole" H 2750 1900 50  0001 C CNN
+F 2 "Custom_FP:TactileHole" H 2750 1900 50  0001 C CNN
 F 3 "~" H 2750 1900 50  0001 C CNN
 	1    2750 1900
@@
 F 0 "H8" H 2900 2196 50  0000 L CNN
 F 1 "MountingHole" H 2900 2105 50  0000 L CNN
-F 2 "CustomLib:TactileHole" H 2800 2150 50  0001 C CNN
+F 2 "Custom_FP:TactileHole" H 2800 2150 50  0001 C CNN
 F 3 "~" H 2800 2150 50  0001 C CNN
 	1    2800 2150
@@
 F 0 "H4" H 2850 2496 50  0000 L CNN
 F 1 "MountingHole" H 2850 2405 50  0000 L CNN
-F 2 "CustomLib:TactileHole" H 2750 2450 50  0001 C CNN
+F 2 "Custom_FP:TactileHole" H 2750 2450 50  0001 C CNN
 F 3 "~" H 2750 2450 50  0001 C CNN
 	1    2750 2450
@@
 F 0 "H5" H 2850 2796 50  0000 L CNN
 F 1 "MountingHole" H 2850 2705 50  0000 L CNN
-F 2 "CustomLib:TactileHole" H 2750 2750 50  0001 C CNN
+F 2 "Custom_FP:TactileHole" H 2750 2750 50  0001 C CNN
 F 3 "~" H 2750 2750 50  0001 C CNN
 	1    2750 2750
@@
 F 0 "H1" H 2800 3096 50  0000 L CNN
 F 1 "MountingHole" H 2800 3005 50  0000 L CNN
-F 2 "CustomLib:TactileHole" H 2700 3050 50  0001 C CNN
+F 2 "Custom_FP:TactileHole" H 2700 3050 50  0001 C CNN
 F 3 "~" H 2700 3050 50  0001 C CNN
 	1    2700 3050
@@
 F 0 "H2" H 2800 3346 50  0000 L CNN
 F 1 "MountingHole" H 2800 3255 50  0000 L CNN
-F 2 "CustomLib:TactileHole" H 2700 3300 50  0001 C CNN
+F 2 "Custom_FP:TactileHole" H 2700 3300 50  0001 C CNN
 F 3 "~" H 2700 3300 50  0001 C CNN
 	1    2700 3300
@@
 F 0 "H7" H 2850 3846 50  0000 L CNN
 F 1 "MountingHole" H 2850 3755 50  0000 L CNN
-F 2 "CustomLib:TactileHole" H 2750 3800 50  0001 C CNN
+F 2 "Custom_FP:TactileHole" H 2750 3800 50  0001 C CNN
 F 3 "~" H 2750 3800 50  0001 C CNN
 	1    2750 3800
@@
 F 0 "H6" H 2850 3596 50  0000 L CNN
 F 1 "MountingHole" H 2850 3505 50  0000 L CNN
-F 2 "CustomLib:TactileHole" H 2750 3550 50  0001 C CNN
+F 2 "Custom_FP:TactileHole" H 2750 3550 50  0001 C CNN
 F 3 "~" H 2750 3550 50  0001 C CNN
 	1    2750 3550
