File: Core/Core.kicad_sch (KiCad schematic)
At the start: 15 parts, among them U10 TL072, U11 TL072, U12 TL072, U13 TL072, U17 74HC595, U19 74HC595, U2 DG408, U20 74HC595, U3 DG408, U4 DG408, U5 DG408, U6 DG408, U7 DG408, U8 DG408, U9 DG408

Commit message: Update sheet metadata
Other:
- company: (none) -> GuavTek
- title: (none) -> M2IDI_CORE
Changed lines of the file:
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@@
 (kicad_sch (version 20230121) (generator eeschema)
   (paper "A4")
+  (title_block
+    (title "M2IDI_CORE")
+    (date "2023-04-19")
+    (rev "1.1")
+    (company "GuavTek")
+  )
   (junction (at 118.11 149.86) (diameter 0) (color 0 0 0 0)
   )

Commit message: Fix metadata
Other:
- title: M2IDI_CORE -> M2IDI - TANGLE CORE
Changed lines of the file:
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@@
   (paper "A4")
   (title_block
-    (title "M2IDI_CORE")
+    (title "M2IDI - TANGLE CORE")
     (date "2023-04-19")
     (rev "1.1")
