File: Core/Power.kicad_sch (KiCad schematic)
At the start: 50 parts, among them J21 Conn_02x08_Odd_Even, Q1 BSS84, Q2 2N7002, Q3 BSS84, U10 TL072, U11 TL072, U12 TL072, U13 TL072, U18 MIC5504-3.3YM5

Commit message: Update sheet metadata
Other:
- company: (none) -> GuavTek
- title: (none) -> M2IDI_CORE
Changed lines of the file:
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@@
 (kicad_sch (version 20230121) (generator eeschema)
   (paper "A4")
+  (title_block
+    (title "M2IDI_CORE")
+    (date "2023-04-19")
+    (rev "1.1")
+    (company "GuavTek")
+  )
   (junction (at 237.49 110.49) (diameter 0) (color 0 0 0 0)
   )

Commit message: Fix metadata
Other:
- title: M2IDI_CORE -> M2IDI - TANGLE CORE
Changed lines of the file:
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@@
   (paper "A4")
   (title_block
-    (title "M2IDI_CORE")
+    (title "M2IDI - TANGLE CORE")
     (date "2023-04-19")
     (rev "1.1")
